Commit message: Added RViz launch and ROS2 MoveIt integration (with panda from AndrejOrsula github)

File: panda_description/urdf/panda.urdf (robot description, URDF)
Before this commit: robot panda, 14 links, 13 joints
Links:
- added link wrist_camera_link, mass 0.05
Joints:
- added joint wrist_camera_joint: type fixed, parent panda_link8, child wrist_camera_link, origin xyz=0.06 0 0.02 rpy=0 -1.5708 0.7854

File: panda_description/urdf/panda.urdf.xacro (robot description, xacro)
@@ -32,6 +32,6 @@
   <!-- Flag to enable ros2 controllers for manipulator -->
   <xacro:arg name="ros2_control" default="true"/>
-  <!-- The ros2_control plugin that should be loaded for the manipulator ('fake', 'ign', 'real' or custom) -->
-  <xacro:arg name="ros2_control_plugin" default="ign"/>
+  <!-- The ros2_control plugin that should be loaded for the manipulator ('fake', 'gz', 'real' or custom) -->
+  <xacro:arg name="ros2_control_plugin" default="gz"/>
   <!-- The output control command interface provided by ros2_control ('position', 'velocity', 'effort' or certain combinations 'position,velocity') -->
   <xacro:arg name="ros2_control_command_interface" default="effort"/>
@@ -91,8 +91,32 @@
     />
   </xacro:if>
-  <!-- Gazebo - ROS 2 control (Ignition) -->
+  <!-- Wrist camera -->
+  <link name="wrist_camera_link">
+    <inertial>
+      <mass value="0.05"/>
+      <inertia ixx="1e-5" ixy="0" ixz="0" iyy="1e-5" iyz="0" izz="1e-5"/>
+    </inertial>
+  </link>
+  <joint name="wrist_camera_joint" type="fixed">
+    <parent link="${prefix_arm}link8"/>
+    <child link="wrist_camera_link"/>
+    <origin xyz="0.06 0 0.02" rpy="0 -1.5708 0.7854"/>
+  </joint>
+  <gazebo reference="wrist_camera_link">
+    <sensor name="wrist_camera" type="rgbd_camera">
+      <topic>wrist_camera</topic>
+      <camera>
+        <horizontal_fov>1.047</horizontal_fov>
+        <image><width>640</width><height>480</height></image>
+        <clip><near>0.05</near><far>2.0</far></clip>
+      </camera>
+      <update_rate>15</update_rate>
+      <always_on>true</always_on>
+    </sensor>
+  </gazebo>
+  <!-- Gazebo - ROS 2 control -->
   <xacro:if value="$(arg ros2_control)">
-    <xacro:if value="${'ign' in '$(arg ros2_control_plugin)'}">
-      <xacro:ign_ros2_control controller_parameters="$(arg ros2_controller_parameters)"/>
+    <xacro:if value="${'gz' in '$(arg ros2_control_plugin)'}">
+      <xacro:gz_ros2_control controller_parameters="$(arg ros2_controller_parameters)"/>
     </xacro:if>
   </xacro:if>
