Commit message: Panda arm  in scene implemented

File: panda_description/urdf/panda.urdf.xacro (robot description, xacro)
@@ -48,6 +48,6 @@
   <!-- Origin of arm in the world -->
   <xacro:property name="world_name" value="world"/>
-  <xacro:property name="origin_xyz" value="0 0 0"/>
-  <xacro:property name="origin_rpy" value="0 0 0"/>
+  <xacro:property name="origin_xyz" value="1.0 0 1.01"/>
+  <xacro:property name="origin_rpy" value="0 0 3.14159"/>
   <!-- Offset of gripper with respect to wrist flange -->
   <xacro:property name="gripper_offset_xyz" value="0 0 0"/>

File: panda_description/urdf/panda_gripper.xacro (robot description, xacro)
@@ -26,5 +26,5 @@
   <xacro:property name="joint_finger1_friction" value="0.4"/>
   <xacro:property name="link_finger1_name" value="leftfinger"/>
-  <xacro:property name="link_finger1_mu" value="1.13"/>
+  <xacro:property name="link_finger1_mu" value="10.0"/>
   <xacro:property name="link_finger1_mesh_offset" value="0 0 0"/>
   <xacro:property name="joint_finger2_name" value="finger_joint2"/>
@@ -40,5 +40,5 @@
   <xacro:property name="joint_finger2_friction" value="0.4"/>
   <xacro:property name="link_finger2_name" value="rightfinger"/>
-  <xacro:property name="link_finger2_mu" value="1.13"/>
+  <xacro:property name="link_finger2_mu" value="10.0"/>
   <xacro:property name="link_finger2_mesh_offset" value="0 0 ${pi}"/>
   <xacro:property name="ee_name" value="hand_tcp"/>
@@ -125,4 +125,13 @@
     mesh_offset_rpy="${link_finger2_mesh_offset}"
     />
+    <!-- Stiff, high-friction contact on fingers so grasped objects don't slip -->
+    <gazebo reference="${prefix}${link_finger1_name}">
+      <kp>1e8</kp>
+      <kd>1</kd>
+    </gazebo>
+    <gazebo reference="${prefix}${link_finger2_name}">
+      <kp>1e8</kp>
+      <kd>1</kd>
+    </gazebo>
     <!-- End effector -->
     <xacro:panda_virtual_link
